Commit message: complete robot driving sim in gazebo, create new multi-launch file, and clean up some mistakes in the URDF

File: carr-e-2/description/robot.urdf.xacro (robot description, xacro)
@@ -1,6 +1,8 @@
 <?xml version="1.0"?>
 <robot xmlns:xacro="http://www.ros.org/wiki/xacro"  name="robot">
-    <xacro:include filename="inertial_macros.xacro" />
-    <xacro:include filename="colors.xacro" />
-    <xacro:include filename="robot_core.xacro" />
+	<include filename="inertial_macros.xacro" />
+	<include filename="colors.xacro" />
+	<include filename="robot_core_sim.xacro" />
+	<include filename="gazebo_control.xacro" />
+	<xacro:include filename="robot_core.xacro" />
 </robot>

File: carr-e-2/description/robot_core.xacro (robot description, xacro)
@@ -1,7 +1,8 @@
 <?xml version="1.0"?>
-<robot xmlns:xacro="http://www.ros.org/wiki/xacro" name="robot">
-    <link name="base_link">
+<robot xmlns:xacro="http://www.ros.org/wiki/xacro">
+	<!-- BASE LINK -->
+	<link name="base_link">
 	</link>
-	<!-- CHASSIS -->
+	<!-- CHASSIS LINK -->
 	<joint name="chassis_joint" type="fixed">
 		<parent link="base_link" />
@@ -11,106 +12,87 @@
 	<link name="chassis">
 		<visual>
+			<origin xyz="0.15 0 0.075" />
+			<geometry>
+				<box size="0.3 0.3 0.15" />
+			</geometry>
+			<material name="white" />
+		</visual>
+		<collision>
+			<origin xyz="0.15 0 0.075" />
+			<geometry>
+				<box size="0.3 0.3 0.15" />
+			</geometry>
+		</collision>
+		<inertial_box mass="0.5" x="0.3" y="0.3" z="0.15">
 			<origin xyz="0.15 0 0.075" rpy="0 0 0" />
-			<geometry>
-				<box size="0.3 0.3 0.15">
-				</box>
-			</geometry>
-			<material name="white">
-			</material>
-		</visual>
-        <collision>
-			<origin xyz="0.15 0 0.075" rpy="0 0 0" />
-			<geometry>
-				<box size="0.3 0.3 0.15">
-				</box>
-			</geometry>
-			<material name="white">
-			</material>
-		</collision>
-        <xacro:inertial_box mass="0.5" x="0.3" y="0.3" z="0.15">
-            <origin xyz="0.15 0 0.075" rpy="0 0 0"/>
-        </xacro:inertial_box>
+		</inertial_box>
 	</link>
+	<!-- LEFT WHEEL LINK -->
 	<joint name="left_wheel_joint" type="continuous">
 		<parent link="base_link" />
 		<child link="left_wheel" />
-		<!-- rotate -pi/2 about x-axis -->
 		<origin xyz="0 0.175 0" rpy="-${pi/2} 0 0" />
-		<!-- rotate about z=1 -->
 		<axis xyz="0 0 1" />
-        <xacro:inertial_cylinder mass="0.1" length="0.05" radius="0.05">
-            <origin xyz="0 0 0" rpy="0 0 0"/>
-        </xacro:inertial_cylinder>
 	</joint>
-	<!-- WHEELS -->
 	<link name="left_wheel">
 		<visual>
 			<geometry>
-				<cylinder length="0.04" radius="0.05">
-				</cylinder>
+				<cylinder radius="0.05" length="0.04" />
 			</geometry>
-			<material name="blue">
-			</material>
+			<material name="blue" />
 		</visual>
-        <collision>
+		<collision>
 			<geometry>
-				<cylinder length="0.04" radius="0.05">
-				</cylinder>
+				<cylinder radius="0.05" length="0.04" />
 			</geometry>
-			<material name="blue">
-			</material>
 		</collision>
+		<inertial_cylinder mass="0.1" length="0.04" radius="0.05">
+			<origin xyz="0 0 0" rpy="0 0 0" />
+		</inertial_cylinder>
 	</link>
+	<!-- RIGHT WHEEL LINK -->
 	<joint name="right_wheel_joint" type="continuous">
 		<parent link="base_link" />
 		<child link="right_wheel" />
-		<!-- rotate pi/2 about x-axis -->
 		<origin xyz="0 -0.175 0" rpy="${pi/2} 0 0" />
-		<!-- rotate about z=-1 -->
 		<axis xyz="0 0 -1" />
-        <xacro:inertial_cylinder mass="0.1" length="0.05" radius="0.05">
-            <origin xyz="0 0 0" rpy="0 0 0"/>
-        </xacro:inertial_cylinder>
 	</joint>
 	<link name="right_wheel">
 		<visual>
 			<geometry>
-				<cylinder length="0.04" radius="0.05">
-				</cylinder>
+				<cylinder radius="0.05" length="0.04" />
 			</geometry>
-			<material name="blue">
-			</material>
+			<material name="blue" />
 		</visual>
-        <collision>
+		<collision>
 			<geometry>
-				<cylinder length="0.04" radius="0.05">
-				</cylinder>
+				<cylinder radius="0.05" length="0.04" />
 			</geometry>
-			<material name="blue">
-			</material>
 		</collision>
+		<inertial_cylinder mass="0.1" length="0.04" radius="0.05">
+			<origin xyz="0 0 0" rpy="0 0 0" />
+		</inertial_cylinder>
 	</link>
-	<!-- CASTER WHEEL -->
+	<!-- CASTER WHEEL LINK -->
 	<joint name="caster_wheel_joint" type="fixed">
-        <parent link="chassis"></parent>
-        <child link="caster_wheel"></child>
-        <origin xyz="0.24 0 0" rpy="0 0 0"></origin>
+		<parent link="chassis" />
+		<child link="caster_wheel" />
+		<origin xyz="0.24 0 0" />
 	</joint>
-    <link name="caster_wheel">
-        <visual>
-            <geometry>
-                <sphere radius="0.05"></sphere>
-            </geometry>
-            <material name="black"></material>
-        </visual>
-        <collision>
-            <geometry>
-                <sphere radius="0.05"></sphere>
-            </geometry>
-            <material name="black"></material>
-        </collision>
-        <xacro:inertial_sphere mass="0.1" radius="0.05">
-            <origin xyz="0 0 0" rpy="0 0 0"/>
-        </xacro:inertial_sphere>
-    </link>
+	<link name="caster_wheel">
+		<visual>
+			<geometry>
+				<sphere radius="0.05" />
+			</geometry>
+			<material name="black" />
+		</visual>
+		<collision>
+			<geometry>
+				<sphere radius="0.05" />
+			</geometry>
+		</collision>
+		<inertial_sphere mass="0.1" radius="0.05">
+			<origin xyz="0 0 0" rpy="0 0 0" />
+		</inertial_sphere>
+	</link>
 </robot>
