Commit message: add lidar in both ros and gazbo simulation

File: carr-e-2/description/colors.xacro (robot description, xacro)
@@ -13,3 +13,6 @@
     <color rgba="0.2 0.2 1 1"/>
 </material>
+<material name="red">
+    <color rgba="1 0 0 1"/>
+</material>
 </robot>

File: carr-e-2/description/robot.urdf.xacro (robot description, xacro)
@@ -6,3 +6,4 @@
 	<xacro:include filename="gazebo_control.xacro" />
 	<xacro:include filename="robot_core.xacro" />
+	<xacro:include filename="lidar.xacro" />
 </robot>

File: carr-e-2/description/robot_core_sim.xacro (robot description, xacro)
@@ -24,3 +24,11 @@
         <mu2 value="0.001"/>
     </gazebo>
+    <!-- GAZEBO LIDAR -->
+    <gazebo reference="laser_frame">
+        <material>
+            Gazebo/Red
+        </material>
+        <!-- <mu1 value="0.001"/>
+        <mu2 value="0.001"/> -->
+    </gazebo>
 </robot>
