Commit message: add camera simulation

File: carr-e-2/description/lidar.xacro (robot description, xacro)
@@ -1,11 +1,14 @@
 <?xml version="1.0"?>
 <robot xmlns:xacro="http://www.ros.org/wiki/xacro">
-    <joint name="laser_joint" type="fixed">
-        <parent link="chassis"></parent>
-        <child link="laser_frame"></child>
-        <origin xyz="0.1 0 0.175" rpy="0 0 0"></origin>
-    </joint>
-    <link name="laser_frame">
-        	<visual>
+	<joint name="laser_joint" type="fixed">
+		<parent link="chassis">
+		</parent>
+		<child link="laser_frame">
+		</child>
+		<origin xyz="0.1 0 0.175" rpy="0 0 0">
+		</origin>
+	</joint>
+	<link name="laser_frame">
+		<visual>
 			<geometry>
 				<cylinder radius="0.05" length="0.04" />
@@ -21,33 +24,59 @@
 			<origin xyz="0 0 0" rpy="0 0 0" />
 		</inertial_cylinder>
-    </link>
-    <gazebo reference="laser_frame">
-    <sensor name="laser" type="ray">
-    <pose>0 0 0 0 0 0</pose>
-    <visualize>true</visualize>
-    <update_rate>10</update_rate>
-    <ray>
-        <scan>
-        <horizontal>
-            <samples>360</samples>
-            <resolution>1</resolution>
-            <min_angle>-3.14</min_angle>
-            <max_angle>3.14</max_angle>
-        </horizontal>
-        </scan>
-        <range>
-        <min>0.3</min>
-        <max>12</max>
-        <resolution>0.01</resolution>
-        </range>
-        </ray>
-        <plugin name="laser_controller" filename="libgazebo_ros_ray_sensor.so">
-        <ros>
-        <argument>~/out:=scan</argument>
-        </ros>
-        <output_type>sensor_msgs/LaserScan</output_type>
-        <frame_name>laser_frame</frame_name>
-        </plugin>
-    </sensor>
-    </gazebo>
+	</link>
+	<gazebo reference="laser_frame">
+		<sensor name="laser" type="ray">
+			<pose>
+				0 0 0 0 0 0
+			</pose>
+			<visualize>
+				true
+			</visualize>
+			<update_rate>
+				10
+			</update_rate>
+			<ray>
+				<scan>
+					<horizontal>
+						<samples>
+							360
+						</samples>
+						<resolution>
+							1
+						</resolution>
+						<min_angle>
+							-3.14
+						</min_angle>
+						<max_angle>
+							3.14
+						</max_angle>
+					</horizontal>
+				</scan>
+				<range>
+					<min>
+						0.3
+					</min>
+					<max>
+						12
+					</max>
+					<resolution>
+						0.01
+					</resolution>
+				</range>
+			</ray>
+			<plugin name="laser_controller" filename="libgazebo_ros_ray_sensor.so">
+				<ros>
+					<argument>
+						~/out:=scan
+					</argument>
+				</ros>
+				<output_type>
+					sensor_msgs/LaserScan
+				</output_type>
+				<frame_name>
+					laser_frame
+				</frame_name>
+			</plugin>
+		</sensor>
+	</gazebo>
 </robot>

File: carr-e-2/description/robot.urdf.xacro (robot description, xacro)
@@ -7,3 +7,4 @@
 	<xacro:include filename="robot_core.xacro" />
 	<xacro:include filename="lidar.xacro" />
+	<xacro:include filename="camera.xacro" />
 </robot>

File: carr-e-2/description/robot_core_sim.xacro (robot description, xacro)
@@ -32,3 +32,11 @@
         <mu2 value="0.001"/> -->
     </gazebo>
+    <!-- GAZEBO CAMERA -->
+    <gazebo reference="camera_link">
+        <material>
+            Gazebo/Green
+        </material>
+        <!-- <mu1 value="0.001"/>
+        <mu2 value="0.001"/> -->
+    </gazebo>
 </robot>
