Commit message: fix issues in ros control like wheel collisions and change gazebo to ros simulation frequency to make it smoother

File: carr-e-2/description/robot_core.xacro (robot description, xacro)
@@ -44,5 +44,5 @@
 		<collision>
 			<geometry>
-				<cylinder radius="0.05" length="0.04" />
+				<sphere radius="0.05" />
 			</geometry>
 		</collision>
@@ -67,5 +67,5 @@
 		<collision>
 			<geometry>
-				<cylinder radius="0.05" length="0.04" />
+				<sphere radius="0.05" />
 			</geometry>
 		</collision>

Commit message: finish slam setup but try to make nav2 work

File: carr-e-2/description/robot_core.xacro (robot description, xacro)
@@ -3,4 +3,12 @@
 	<!-- BASE LINK -->
 	<link name="base_link">
+	</link>
+	<!-- BASE FOOTPRINT -->
+	<joint name="base_footprint_joint" type="fixed">
+		<parent link="base_link" />
+		<child link="base_footprint" />
+		<origin xyz="0 0 0" />
+	</joint>
+	<link name="base_footprint">
 	</link>
 	<!-- CHASSIS LINK -->
